Commit message: doesn't work

File: src/my_r2d2/urdf/r2d2.urdf (robot description, URDF)
Before this commit: robot macroed, 17 links, 16 joints
Links:
- added link base_footprint
Joints:
- added joint base_footprint_to_base_link: type fixed, parent base_footprint, child base_link

File: src/my_r2d2/urdf/r2d2.urdf.xacro (robot description, xacro)
@@ -23,4 +23,10 @@
     </inertial>
   </xacro:macro>
+  <link name="base_footprint">
+  </link>
+  <joint name="base_footprint_to_base_link" type="fixed">
+    <parent link="base_footprint"/>
+    <child link="base_link"/>
+  </joint>
   <link name="base_link">
     <visual>
