Commit message: je

File: src/my_r2d2/urdf/r2d2.urdf.xacro (robot description, xacro)
@@ -28,4 +28,5 @@
     <parent link="base_footprint"/>
     <child link="base_link"/>
+    <origin xyz="0 0 0.45"/>
   </joint>
   <link name="base_link">

Commit message: ...

File: src/my_r2d2/urdf/r2d2.urdf.xacro (robot description, xacro)
@@ -8,4 +8,5 @@
   <xacro:property name="wheeldiam" value="0.07" />
   <xacro:property name="pi" value="3.1415" />
+  <xacro:property name="reflect" value="1" />
   <material name="blue">
     <color rgba="0 0 0.8 1"/>
@@ -23,25 +24,45 @@
     </inertial>
   </xacro:macro>
+  <link name="eye">
+  </link>
+    <joint name="eye_joint" type="fixed">
+      <parent link="lense"/>
+      <child link="eye"/>
+      <origin xyz="0 0 0" rpy="-1 1.57 0"/>
+    </joint>
+  <link name="base_link">
+    <visual>
+      <geometry>
+        <cylinder radius="${width}" length="${bodylen}"/>
+      </geometry>
+      <material name="blue"/>
+    </visual>
+    <collision>
+      <geometry>
+        <cylinder radius="${width}" length="${bodylen}"/>
+      </geometry>
+    </collision>
+    <xacro:default_inertial mass="10"/>
+  </link>
+  <link name="lense">
+  <visual>
+  <origin xyz="-0.01 -0.01 0" rpy="0 0 0" />
+      <geometry>
+        <sphere radius="0.03"/>
+      </geometry>
+      <material name="black"/>
+    </visual></link>
   <link name="base_footprint">
   </link>
-  <joint name="base_footprint_to_base_link" type="fixed">
-    <parent link="base_footprint"/>
-    <child link="base_link"/>
-    <origin xyz="0 0 0.45"/>
-  </joint>
-  <link name="base_link">
-    <visual>
-      <geometry>
-        <cylinder radius="${width}" length="${bodylen}"/>
-      </geometry>
-      <material name="blue"/>
-    </visual>
-    <collision>
-      <geometry>
-        <cylinder radius="${width}" length="${bodylen}"/>
-      </geometry>
-    </collision>
-    <xacro:default_inertial mass="10"/>
-  </link>
+    <joint name="foot_joint" type="fixed">
+      <parent link="base_footprint"/>
+      <child link="base_link"/>
+      <origin xyz="0 0 0.44" rpy="0 0 0"/>
+    </joint>
+<joint name="lense_holder" type="fixed">
+      <parent link="box"/>
+      <child link="lense"/>
+      <origin xyz="0 0 0" rpy="0 0 -1"/>
+    </joint>
   <xacro:macro name="wheel" params="prefix suffix reflect">
     <link name="${prefix}_${suffix}_wheel">
@@ -220,16 +241,3 @@
     <origin xyz="${.707*width+0.04} 0 ${.707*width}"/>
   </joint>
-  <link name="eye">
-	<visual>
-      <geometry>
-        <sphere radius="0.03"/>
-      </geometry>
-     <material name="black"/>
-    </visual>
-  </link>
-  <joint name="eye_joint" type="fixed">
-    <parent link="box"/>
-    <child link="eye"/>
-    <origin xyz="0.01 0 0"/>
-  </joint>
 </robot>
